File: Proyecto ZorionX  Nivara/avance del proyecto/borad_zorionx.kicad_sch (KiCad schematic)
At the start: 0 parts

Commit message: Add files via upload
Changed lines of the file:
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@@
+		)
+	)
+	(hierarchical_label "NPN_OUT_2"
+		(shape output)
+		(at 77.47 29.21 0)
+		(fields_autoplaced yes)
+		(effects
+			(font
+				(size 1.27 1.27)
+			)
+			(justify left)
+		)
+	)
+	(hierarchical_label "RU{slash}STOP"
+		(shape input)
+		(at 19.05 80.01 0)
+		(fields_autoplaced yes)
+		(effects
+			(font
+				(size 1.27 1.27)
+			)
+			(justify left)
 		)
 	)
@@
 		(shape input)
 		(at 20.32 68.58 0)
+		(fields_autoplaced yes)
+		(effects
+			(font
+				(size 1.27 1.27)
+			)
+			(justify left)
+		)
+	)
+	(hierarchical_label "NPN_OUT_1"
+		(shape output)
+		(at 77.47 25.4 0)
+		(fields_autoplaced yes)
+		(effects
+			(font
+				(size 1.27 1.27)
+			)
+			(justify left)
+		)
+	)
+	(hierarchical_label "PNP_OUT_2"
+		(shape output)
+		(at 77.47 38.1 0)
 		(fields_autoplaced yes)
 		(effects
@@
 		(fields_autoplaced yes)
 		(effects
+			(font
+				(size 1.27 1.27)
+			)
+			(justify left)
+		)
+	)
+	(hierarchical_label "PNP_OUT_1"
+		(shape output)
+		(at 77.47 34.29 0)
+		(fields_autoplaced yes)
+		(effects
