File: Proyecto ZorionX  Nivara/avance del proyecto/fuente de alimentacion.kicad_sch (KiCad schematic)
At the start: 0 parts

Commit message: Add files via upload
Parts:
- added C1: 10uF 50V, Capacitor_SMD:C_1206_3216Metric, symbol Device:C
- added C2: C, Capacitor_SMD:C_1206_3216Metric, symbol Device:C
- added C3: 100PF, Capacitor_SMD:C_1206_3216Metric, symbol Device:C
- added C4, C5: 22uF, Capacitor_SMD:C_1206_3216Metric, symbol Device:C
- added JP1: SolderJumper_2_Open, symbol Jumper:SolderJumper_2_Open
- added L1: L_Iron_Small, symbol Device:L_Iron_Small
- added R1, R2: 22K 1, Resistor_SMD:R_1206_3216Metric, symbol Device:R
- added TP1, TP2, TP3, TP4: TestPoint, symbol Connector:TestPoint
- added U1: AP63203WU, Package_TO_SOT_SMD:TSOT-23-6, symbol Regulator_Switching:AP63203WU
Connections:
- net +3.3V: now also JP1.1 (A), TP3.1
- new net: C3.1, R1.2, R2.1, TP4.1, U1.1 (FB)
- new net: C2.1, L1.1, U1.5 (SW)
- new net: C2.2, U1.6 (BST)
- new net: C3.2, C4.2, C5.2, JP1.2 (B), L1.2, R1.1, TP2.1
- new net GND: C1.2, C4.1, C5.1, R2.2, U1.4 (GND)
- new net VCC: C1.1, TP1.1, U1.2 (EN), U1.3 (IN)
